Commit message: use stl for collision instead

File: ycb/_prototype.urdf (robot description, URDF)
Before this commit: robot _name, 1 links, 0 joints
Links:
- link base_link: geometry collision mesh filename=_prototype.stl scale=1 1 1; visual mesh filename=_prototype.obj scale=1 1 1

File: ycb/a_colored_wood_blocks.urdf (robot description, URDF)
Before this commit: robot a_colored_wood_blocks, 1 links, 0 joints
Links:
- link base_link: geometry collision mesh filename=070-a_colored_wood_blocks/google_16k/textured_vhacd.stl scale=1 1 1; visual mesh filename=070-a_colored_wood_blocks/google_16k/textured.obj scale=1 1 1

File: ycb/a_cups.urdf (robot description, URDF)
Before this commit: robot a_cups, 1 links, 0 joints
Links:
- link base_link: geometry collision mesh filename=065-a_cups/google_16k/textured_vhacd.stl scale=1 1 1; visual mesh filename=065-a_cups/google_16k/textured.obj scale=1 1 1

File: ycb/a_lego_duplo.urdf (robot description, URDF)
Before this commit: robot a_lego_duplo, 1 links, 0 joints
Links:
- link base_link: geometry collision mesh filename=073-a_lego_duplo/google_16k/textured_vhacd.stl scale=1 1 1; visual mesh filename=073-a_lego_duplo/google_16k/textured.obj scale=1 1 1

File: ycb/a_marbles.urdf (robot description, URDF)
Before this commit: robot a_marbles, 1 links, 0 joints
Links:
- link base_link: geometry collision mesh filename=063-a_marbles/google_16k/textured_vhacd.stl scale=1 1 1; visual mesh filename=063-a_marbles/google_16k/textured.obj scale=1 1 1

File: ycb/a_toy_airplane.urdf (robot description, URDF)
Before this commit: robot a_toy_airplane, 1 links, 0 joints
Links:
- link base_link: geometry collision mesh filename=072-a_toy_airplane/google_16k/textured_vhacd.stl scale=1 1 1; visual mesh filename=072-a_toy_airplane/google_16k/textured.obj scale=1 1 1

File: ycb/adjustable_wrench.urdf (robot description, URDF)
Before this commit: robot adjustable_wrench, 1 links, 0 joints
Links:
- link base_link: geometry collision mesh filename=042_adjustable_wrench/google_16k/textured_vhacd.stl scale=1 1 1; visual mesh filename=042_adjustable_wrench/google_16k/textured.obj scale=1 1 1

File: ycb/apple.urdf (robot description, URDF)
Before this commit: robot apple, 1 links, 0 joints
Links:
- link base_link: geometry collision mesh filename=013_apple/google_16k/textured_vhacd.stl scale=1 1 1; visual mesh filename=013_apple/google_16k/textured.obj scale=1 1 1

File: ycb/b_colored_wood_blocks.urdf (robot description, URDF)
Before this commit: robot b_colored_wood_blocks, 1 links, 0 joints
Links:
- link base_link: geometry collision mesh filename=070-b_colored_wood_blocks/google_16k/textured_vhacd.stl scale=1 1 1; visual mesh filename=070-b_colored_wood_blocks/google_16k/textured.obj scale=1 1 1

File: ycb/b_cups.urdf (robot description, URDF)
Before this commit: robot b_cups, 1 links, 0 joints
Links:
- link base_link: geometry collision mesh filename=065-b_cups/google_16k/textured_vhacd.stl scale=1 1 1; visual mesh filename=065-b_cups/google_16k/textured.obj scale=1 1 1

File: ycb/b_lego_duplo.urdf (robot description, URDF)
Before this commit: robot b_lego_duplo, 1 links, 0 joints
Links:
- link base_link: geometry collision mesh filename=073-b_lego_duplo/google_16k/textured_vhacd.stl scale=1 1 1; visual mesh filename=073-b_lego_duplo/google_16k/textured.obj scale=1 1 1

File: ycb/b_marbles.urdf (robot description, URDF)
Before this commit: robot b_marbles, 1 links, 0 joints
Links:
- link base_link: geometry collision mesh filename=063-b_marbles/google_16k/textured_vhacd.stl scale=1 1 1; visual mesh filename=063-b_marbles/google_16k/textured.obj scale=1 1 1

File: ycb/b_toy_airplane.urdf (robot description, URDF)
Before this commit: robot b_toy_airplane, 1 links, 0 joints
Links:
- link base_link: geometry collision mesh filename=072-b_toy_airplane/google_16k/textured_vhacd.stl scale=1 1 1; visual mesh filename=072-b_toy_airplane/google_16k/textured.obj scale=1 1 1

File: ycb/banana.urdf (robot description, URDF)
Before this commit: robot banana, 1 links, 0 joints
Links:
- link base_link: geometry collision mesh filename=011_banana/google_16k/textured_vhacd.stl scale=1 1 1; visual mesh filename=011_banana/google_16k/textured.obj scale=1 1 1

File: ycb/baseball.urdf (robot description, URDF)
Before this commit: robot baseball, 1 links, 0 joints
Links:
- link base_link: geometry collision mesh filename=055_baseball/google_16k/textured_vhacd.stl scale=1 1 1; visual mesh filename=055_baseball/google_16k/textured.obj scale=1 1 1

File: ycb/bleach_cleanser.urdf (robot description, URDF)
Before this commit: robot bleach_cleanser, 1 links, 0 joints
Links:
- link base_link: geometry collision mesh filename=021_bleach_cleanser/google_16k/textured_vhacd.stl scale=1 1 1; visual mesh filename=021_bleach_cleanser/google_16k/textured.obj scale=1 1 1

File: ycb/bowl.urdf (robot description, URDF)
Before this commit: robot bowl, 1 links, 0 joints
Links:
- link base_link: geometry collision mesh filename=024_bowl/google_16k/textured_vhacd.stl scale=1 1 1; visual mesh filename=024_bowl/google_16k/textured.obj scale=1 1 1

File: ycb/c_cups.urdf (robot description, URDF)
Before this commit: robot c_cups, 1 links, 0 joints
Links:
- link base_link: geometry collision mesh filename=065-c_cups/google_16k/textured_vhacd.stl scale=1 1 1; visual mesh filename=065-c_cups/google_16k/textured.obj scale=1 1 1

File: ycb/c_lego_duplo.urdf (robot description, URDF)
Before this commit: robot c_lego_duplo, 1 links, 0 joints
Links:
- link base_link: geometry collision mesh filename=073-c_lego_duplo/google_16k/textured_vhacd.stl scale=1 1 1; visual mesh filename=073-c_lego_duplo/google_16k/textured.obj scale=1 1 1

File: ycb/c_toy_airplane.urdf (robot description, URDF)
Before this commit: robot c_toy_airplane, 1 links, 0 joints
Links:
- link base_link: geometry collision mesh filename=072-c_toy_airplane/google_16k/textured_vhacd.stl scale=1 1 1; visual mesh filename=072-c_toy_airplane/google_16k/textured.obj scale=1 1 1
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