Commit message: update CoACD meshes

File: ycb/a_colored_wood_blocks.urdf (robot description, URDF)
Before this commit: robot a_colored_wood_blocks, 1 links, 0 joints
Links:
- link base_link: geometry collision mesh filename=a_colored_wood_blocks/textured_coacd_0.stl scale=1 1 1; collision mesh filename=a_colored_wood_blocks/textured_coacd_1.stl scale=1 1 1

File: ycb/a_cups.urdf (robot description, URDF)
Before this commit: robot a_cups, 1 links, 0 joints
Links:
- link base_link: geometry collision mesh filename=a_cups/textured_coacd_0.stl scale=1 1 1; collision mesh filename=a_cups/textured_coacd_1.stl scale=1 1 1

File: ycb/a_lego_duplo.urdf (robot description, URDF)
Before this commit: robot a_lego_duplo, 1 links, 0 joints
Links:
- link base_link: geometry collision mesh filename=a_lego_duplo/textured_coacd_0.stl scale=1 1 1; collision mesh filename=a_lego_duplo/textured_coacd_1.stl scale=1 1 1

File: ycb/a_marbles.urdf (robot description, URDF)
Before this commit: robot a_marbles, 1 links, 0 joints
Links:
- link base_link: geometry collision mesh filename=a_marbles/textured_coacd_0.stl scale=1 1 1; collision mesh filename=a_marbles/textured_coacd_1.stl scale=1 1 1

File: ycb/a_toy_airplane.urdf (robot description, URDF)
Before this commit: robot a_toy_airplane, 1 links, 0 joints
Links:
- link base_link: geometry collision mesh filename=a_toy_airplane/textured_coacd_0.stl scale=1 1 1; collision mesh filename=a_toy_airplane/textured_coacd_1.stl scale=1 1 1

File: ycb/adjustable_wrench.urdf (robot description, URDF)
Before this commit: robot adjustable_wrench, 1 links, 0 joints
Links:
- link base_link: geometry collision mesh filename=adjustable_wrench/textured_coacd_0.stl scale=1 1 1; collision mesh filename=adjustable_wrench/textured_coacd_1.stl scale=1 1 1

File: ycb/apple.urdf (robot description, URDF)
Before this commit: robot apple, 1 links, 0 joints
Links:
- link base_link: geometry collision mesh filename=apple/textured_coacd_0.stl scale=1 1 1; collision mesh filename=apple/textured_coacd_1.stl scale=1 1 1

File: ycb/b_colored_wood_blocks.urdf (robot description, URDF)
Before this commit: robot b_colored_wood_blocks, 1 links, 0 joints
Links:
- link base_link: geometry collision mesh filename=b_colored_wood_blocks/textured_coacd_0.stl scale=1 1 1; collision mesh filename=b_colored_wood_blocks/textured_coacd_1.stl scale=1 1 1

File: ycb/b_cups.urdf (robot description, URDF)
Before this commit: robot b_cups, 1 links, 0 joints
Links:
- link base_link: geometry collision mesh filename=b_cups/textured_coacd_0.stl scale=1 1 1; collision mesh filename=b_cups/textured_coacd_1.stl scale=1 1 1

File: ycb/b_lego_duplo.urdf (robot description, URDF)
Before this commit: robot b_lego_duplo, 1 links, 0 joints
Links:
- link base_link: geometry collision mesh filename=b_lego_duplo/textured_coacd_0.stl scale=1 1 1; collision mesh filename=b_lego_duplo/textured_coacd_1.stl scale=1 1 1

File: ycb/b_marbles.urdf (robot description, URDF)
Before this commit: robot b_marbles, 1 links, 0 joints
Links:
- link base_link: geometry collision mesh filename=b_marbles/textured_coacd_0.stl scale=1 1 1; visual mesh filename=b_marbles/textured.obj scale=1 1 1

File: ycb/b_toy_airplane.urdf (robot description, URDF)
Before this commit: robot b_toy_airplane, 1 links, 0 joints
Links:
- link base_link: geometry collision mesh filename=b_toy_airplane/textured_coacd_0.stl scale=1 1 1; collision mesh filename=b_toy_airplane/textured_coacd_1.stl scale=1 1 1

File: ycb/banana.urdf (robot description, URDF)
Before this commit: robot banana, 1 links, 0 joints
Links:
- link base_link: geometry collision mesh filename=banana/textured_coacd_0.stl scale=1 1 1; collision mesh filename=banana/textured_coacd_1.stl scale=1 1 1

File: ycb/baseball.urdf (robot description, URDF)
Before this commit: robot baseball, 1 links, 0 joints
Links:
- link base_link: geometry collision mesh filename=baseball/textured_coacd_0.stl scale=1 1 1; visual mesh filename=baseball/textured.obj scale=1 1 1

File: ycb/bleach_cleanser.urdf (robot description, URDF)
Before this commit: robot bleach_cleanser, 1 links, 0 joints
Links:
- link base_link: geometry collision mesh filename=bleach_cleanser/textured_coacd_0.stl scale=1 1 1; collision mesh filename=bleach_cleanser/textured_coacd_1.stl scale=1 1 1

File: ycb/bowl.urdf (robot description, URDF)
Before this commit: robot bowl, 1 links, 0 joints
Links:
- link base_link: geometry collision mesh filename=bowl/textured_coacd_0.stl scale=1 1 1; collision mesh filename=bowl/textured_coacd_1.stl scale=1 1 1

File: ycb/c_cups.urdf (robot description, URDF)
Before this commit: robot c_cups, 1 links, 0 joints
Links:
- link base_link: geometry collision mesh filename=c_cups/textured_coacd_0.stl scale=1 1 1; collision mesh filename=c_cups/textured_coacd_1.stl scale=1 1 1

File: ycb/c_lego_duplo.urdf (robot description, URDF)
Before this commit: robot c_lego_duplo, 1 links, 0 joints
Links:
- link base_link: geometry collision mesh filename=c_lego_duplo/textured_coacd_0.stl scale=1 1 1; collision mesh filename=c_lego_duplo/textured_coacd_1.stl scale=1 1 1

File: ycb/c_toy_airplane.urdf (robot description, URDF)
Before this commit: robot c_toy_airplane, 1 links, 0 joints
Links:
- link base_link: geometry collision mesh filename=c_toy_airplane/textured_coacd_0.stl scale=1 1 1; collision mesh filename=c_toy_airplane/textured_coacd_1.stl scale=1 1 1

File: ycb/chain.urdf (robot description, URDF)
Before this commit: robot chain, 1 links, 0 joints
Links:
- link base_link: geometry collision mesh filename=chain/textured_coacd_0.stl scale=1 1 1; collision mesh filename=chain/textured_coacd_1.stl scale=1 1 1
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